File: hardware/MC68000-v5/MC68000.kicad_sch (KiCad schematic)
At the start: 71 parts, among them IC1 MC68681P, J1 Conn_Coaxial_Power, J2 FT232RL board, J3 DUART_OP_PORT, Q1 2N3904, Q2 2N3904, SW1 reset, SW2 SW_SPST, U1 68000D, U10 74LS04, U11 74LS138, U12 628128_DIP32_SSOP32, U13 74LS00, U14 74LS08, U15 28C256, U16 28C256, U17 74LS32, U18 74LS32, U19 EW20200YMY, U2 74LS74, U20 628128_DIP32_SSOP32, U21 DS1813-5, U22 74HC14, U23 74HC14, U24 74HC74, U25 74LS00, U26 74LS00, U29 74LS138, U3 74LS373, U31 DS12887, U32 74LS74, U4 74LS373, U5 74LS373, U6 74LS245, U7 74LS245, U8 74LS32, U9 74LS04, Y1 16MHz, Y2 3.6864 MHz

Commit message: minor change to v5 version
Connections:
- net DUART_OR_LCD is gone; now on net DUART_LCD_ACK: U10.1, U13.3
- net +5V: no longer U14.4, U14.5
- net DUART_LCD_ACK: no longer U10.2, U13.4
- net /IO_ACK: now also U14.4; no longer U25.13
- net at R18.2: now also D2.2 (A); no longer D2.1 (K)
- net /CS_LED: now reaches U29.7 (O7)
- net /CS_LED: now also D2.1 (K), U14.5; no longer D2.2 (A)
- net /IO_ACK_ALL: now reaches U14.6
- net /IO_ACK_ALL: now also U25.13
- net IO_ANY renamed DURAT_LCD_RTS_ACK
- new net /DUART_LCD_ACK: U10.2, U13.4
- no-connect marks 33 -> 32

Commit message: rewiring 1
Parts:
- U24: renamed from U32; footprint Package_DIP:DIP-20_W7.62mm -> (none)
- renumbered U2 to U24
Changed lines of the file:
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@@
 		(in_pos_files yes)
 		(dnp no)
-		(property "Reference" "U2"
+		(property "Reference" "U24"
 			(at 392.43 365.2519 0)
 			(show_name no)
@@
 			(project "MC68000"
 				(path "/5c69547b-40ff-41db-a8db-5638c055b360"
-					(reference "U2")
+					(reference "U24")
 					(unit 3)
 				)
@@
 		(dnp no)
 		(fields_autoplaced yes)
-		(property "Reference" "U32"
+		(property "Reference" "U24"
 			(at 189.23 324.486 0)
 			(show_name no)
@@
 			)
 		)
-		(property "Footprint" "Package_DIP:DIP-20_W7.62mm"
+		(property "Footprint" ""
 			(at 189.23 332.486 0)
 			(hide yes)
@@
 			)
 		)
-		(property "Datasheet" ""
+		(property "Datasheet" "https://www.ti.com/lit/ds/symlink/sn74ls74a.pdf"
 			(at 189.23 332.486 0)
 			(hide yes)
@@
 			)
 		)
-		(property "Description" "v4 address-overlay TTL logic"
+		(property "Description" "Dual D Flip-flop, Set & Reset"
 			(at 189.23 332.486 0)
 			(hide yes)
@@
 			(project "MC68000"
 				(path "/5c69547b-40ff-41db-a8db-5638c055b360"
-					(reference "U32")
+					(reference "U24")
 					(unit 1)
 				)
