File: hardware/MC68000-v5/.history/MC68000.kicad_sch (KiCad schematic)
At the start: 69 parts, among them IC1 MC68681P, J1 Conn_Coaxial_Power, J2 FT232RL board, J3 DUART_OP_PORT, Q1 2N3904, Q2 2N3904, SW1 reset, SW2 SW_SPST, U1 68000D, U10 74LS04, U11 74LS138, U12 628128_DIP32_SSOP32, U13 74LS00, U14 74LS08, U15 28C256, U16 28C256, U17 74LS32, U18 74LS32, U19 EW20200YMY, U2 74LS74, U20 628128_DIP32_SSOP32, U21 DS1813-5, U22 74HC14, U23 74HC14, U24 74HC74, U25 74LS00, U26 74LS00, U29 74LS138, U3 74LS373, U31 DS12887, U32 74LS74, U4 74LS373, U5 74LS373, U6 74LS245, U7 74LS245, U8 74LS32, U9 74LS04, Y1 16MHz, Y2 3.6864 MHz

Commit message: rewiring 1
Parts:
- removed unit 1 of U26
- removed unit 3 of U8
- added C11: 100n, Capacitor_THT:C_Disc_D3.0mm_W2.0mm_P2.50mm, symbol Device:C
- added R20: 4.7K, Resistor_THT:R_Axial_DIN0207_L6.3mm_D2.5mm_P7.62mm_Horizontal, symbol Device:R
- added unit 4 of U26
- added unit 2 of U9
- U14: footprint (none) -> Package_DIP:DIP-14_W7.62mm
- U17: footprint Package_DIP:DIP-14_W7.62mm -> (none)
- U24: renamed from U32; footprint Package_DIP:DIP-20_W7.62mm -> (none)
- renumbered U2 to U24
Connections:
- net MEM_PAGE is gone; now on net 0x530000–0x53FFFF: U29.12 (O3)
- net +5V: now also U24.1 (~{R}), U24.14 (VCC), U25.10, U25.9, U26.10, U26.9, U9.13, C11.1, R20.1, U26.12, U26.13; no longer U10.11, U18.12, U18.13
- net GND: now also U17.10, U17.12, U17.13, U17.4, U17.5, U17.9, U24.7 (GND), C11.2
- net LCD_READY: no longer U17.5
- net OVL: now also U14.13, U26.2
- net OVL_D: now also U14.11
- net ROM_SELECT: now also U10.10, U25.1, U25.4; no longer U17.1
- net R/W: now also U18.10
- net /AS: now also U17.1
- net /CS_DUART: now also U8.12; no longer U14.4
- net /CS_LCD: now also U13.2
- net /CS_ROM_H: now also U25.6; no longer U14.11
- net /CS_ROM_L: now also U25.3
- net /CS_RTC: now also U13.5; no longer U10.1
- net /DTACK: now also U17.3; no longer U10.4
- net /LDS: now also U10.13, U18.2, U8.13; no longer U13.10, U14.5, U25.1
- net /RESET: no longer U10.5, U13.5, U14.10, U14.13, U26.10
- net /UDS: now also U18.5, U9.3; no longer U13.13, U25.4
- net /RAM_SELECT: now reaches U18.1, U18.4
- net /RAM_SELECT: now also U13.10, U26.3; no longer U10.6
- net at U26.8: no longer U10.3
- net /HIGH_WIN: now reaches U14.9
- net /HIGH_WIN: now also U11.7 (O7); no longer U25.3
- net /DUART_LCD_ACK: now reaches U10.2
- net /DUART_LCD_ACK: now also U13.4; no longer U17.10
- net /LOW_WIN: now reaches U11.15 (O0)
- net /LOW_WIN: now also U10.9, U18.12; no longer U8.13
- net at R18.2: now also D2.2 (A); no longer D2.1 (K)
- net /CS_LED: now reaches U29.7 (O7)
- net /CS_LED: now also D2.1 (K), U14.5; no longer D2.2 (A)
- net at U25.8: no longer U9.13
- net OVL_KEEP: now reaches U14.12
- net OVL_KEEP: now also U18.8; no longer U25.6
- net DURAT_LCD_RTS_ACK: now reaches U13.6
- net DURAT_LCD_RTS_ACK: now also U10.3; no longer U13.2
- net at U17.11: no longer U26.9
- net at U17.8: no longer U17.13
- net /LOW_ROM_ALIAS: now reaches U18.11
- net /LOW_ROM_ALIAS: now also U14.10
- net at U10.12: now also U25.2
- net at U17.6: no longer U17.9
- net /DUART_ACK: now reaches IC1.9 (DTACK)
- net /DUART_ACK: now also U13.1, R20.2; no longer U25.10
- net MEM_READY: now reaches U13.12
- net MEM_READY: now also U13.13, U13.8; no longer U13.9
- net LOW_WIN: now reaches U10.8
- net LOW_WIN: now also U26.1
- net /DUART_CS: now reaches U8.11
- net /DUART_CS: now also IC1.35 (CS); no longer U14.1
- net /OVL: now reaches U24.6 (~{Q})
- net /OVL: now also U18.13
- net 0x530000–0x53FFFF: now reaches U18.9
- net /CS_ROM_L: no longer names the net of U14.8
- net /CS_ROM_L: now also U10.11
- net DUART_READY: no longer names the net of U9.12
- net DUART_READY: no longer U17.4
- net RAM_SELECT renamed ACK_ANY
- net ACK_ANY: now also U10.5; no longer U17.2
- new net: U25.5, U9.4
- new net DUART_LCD_ACK: U10.1, U13.3
- new net /ACK_SELECT: U10.6, U17.2
- new net /IO_ACK: U10.4, U14.4
- new net /IO_ACK_ALL: U14.6, U25.13
- new net /MEMORY_DTACK: U13.11, U14.1
- new net /MEM_ACK: U14.3, U25.12
- new net /OVL_CONTROL_PAGE: U14.2
- new net /ROM_SELECT: U13.9
- no-connect marks 29 -> 32
